Commit message: Updated Arm Controller

File: my_robot_description/urdf/mobile_base.ros2_control.xacro (robot description, xacro)
@@ -3,10 +3,10 @@
     <ros2_control name="MobileBase" type="system">
         <hardware>
-            <!-- <plugin>mock_components/GenericSystem</plugin>
-            <param name="calculate_dynamics">true</param> -->
-            <plugin>mobile_base_hardware/MobileBaseHardwareInterface</plugin>
+            <plugin>mock_components/GenericSystem</plugin>
+            <param name="calculate_dynamics">true</param>
+            <!-- <plugin>mobile_base_hardware/MobileBaseHardwareInterface</plugin>
             <param name="left_motor_id">10</param>
             <param name="right_motor_id">20</param>
-            <param name="dynamixel_port">/dev/ttyUSB0</param>
+            <param name="dynamixel_port">/dev/ttyUSB0</param> -->
         </hardware>
         <joint name="base_right_wheel_joint">

File: my_robot_description/urdf/my_robot.urdf.xacro (robot description, xacro)
@@ -4,3 +4,10 @@
     <xacro:include filename="mobile_base.xacro" />
     <xacro:include filename="mobile_base.ros2_control.xacro" />
+    <xacro:include filename="arm.xacro"/>
+    <xacro:include filename="arm.ros2_control.xacro"/>
+    <joint name="mobile_base_arm_joint" type="fixed">
+        <parent link="base_link" />
+        <child link="arm_base_link" />
+        <origin xyz="${base_length / 4.0} 0 ${base_height}" rpy="0 0 0" />
+    </joint>
 </robot>
