Commit message: Updated ArmHardwareInterface

File: my_robot_description/urdf/arm.ros2_control.xacro (robot description, xacro)
@@ -3,6 +3,10 @@
     <ros2_control name="Arm" type="system">
         <hardware>
-            <plugin>mock_components/GenericSystem</plugin>
-            <param name="calculate_dynamics">true</param>
+            <!-- <plugin>mock_components/GenericSystem</plugin>
+            <param name="calculate_dynamics">true</param> -->
+            <plugin>arm_hardware/ArmHardwareInterface</plugin>
+            <param name="joint1_motor_id">10</param>
+            <param name="joint2_motor_id">20</param>
+            <param name="dynamixel_port">/dev/ttyUSB0</param>
         </hardware>
         <joint name="arm_joint1">

File: my_robot_description/urdf/arm.xacro (robot description, xacro)
@@ -15,13 +15,4 @@
             <origin xyz="0 0 ${arm_base_height / 2.0}" rpy="0 0 0" />
             <material name="orange" />
-        </visual>
-    </link>
-    <link name="forearm_link">
-        <visual>
-            <geometry>
-                <cylinder radius="${forearm_radius}" length="${forearm_length}" />
-            </geometry>
-            <origin xyz="0 0 ${forearm_length / 2.0}" rpy="0 0 0" />
-            <material name="yellow" />
         </visual>
     </link>

Commit message: Updated Custom ROS2_Controller

File: my_robot_description/urdf/arm.ros2_control.xacro (robot description, xacro)
@@ -3,10 +3,10 @@
     <ros2_control name="Arm" type="system">
         <hardware>
-            <!-- <plugin>mock_components/GenericSystem</plugin>
-            <param name="calculate_dynamics">true</param> -->
-            <plugin>arm_hardware/ArmHardwareInterface</plugin>
+            <plugin>mock_components/GenericSystem</plugin>
+            <param name="calculate_dynamics">true</param>
+            <!-- <plugin>arm_hardware/ArmHardwareInterface</plugin>
             <param name="joint1_motor_id">10</param>
             <param name="joint2_motor_id">20</param>
-            <param name="dynamixel_port">/dev/ttyUSB0</param>
+            <param name="dynamixel_port">/dev/ttyUSB0</param> -->
         </hardware>
         <joint name="arm_joint1">

File: my_robot_description/urdf/arm.xacro (robot description, xacro)
@@ -16,4 +16,29 @@
             <material name="orange" />
         </visual>
+        <collision>
+            <geometry>
+                <box size="${arm_base_length} ${arm_base_width} ${arm_base_height}" />
+            </geometry>
+            <origin xyz="0 0 ${arm_base_height / 2.0}" rpy="0 0 0" />
+        </collision>
+        <xacro:box_inertia m="0.5" x="${arm_base_length}" y="${arm_base_width}" z="${arm_base_height}"
+                           o_xyz="0 0 ${arm_base_height / 2.0}" o_rpy="0 0 0" />
+    </link>
+    <link name="forearm_link">
+        <visual>
+            <geometry>
+                <cylinder radius="${forearm_radius}" length="${forearm_length}" />
+            </geometry>
+            <origin xyz="0 0 ${forearm_length / 2.0}" rpy="0 0 0" />
+            <material name="yellow" />
+        </visual>
+        <collision>
+            <geometry>
+                <cylinder radius="${forearm_radius}" length="${forearm_length}" />
+            </geometry>
+            <origin xyz="0 0 ${forearm_length / 2.0}" rpy="0 0 0" />
+        </collision>
+        <xacro:cylinder_inertia m="0.3" r="${forearm_radius}" l="${forearm_length}"
+                                o_xyz="0 0 ${forearm_length / 2.0}" o_rpy="0 0 0" />
     </link>
     <link name="hand_link">
@@ -25,4 +50,12 @@
             <material name="orange" />
         </visual>
+        <collision>
+            <geometry>
+                <cylinder radius="${hand_radius}" length="${hand_length}" />
+            </geometry>
+            <origin xyz="0 0 ${hand_length / 2.0}" rpy="0 0 0" />
+        </collision>
+        <xacro:cylinder_inertia m="0.3" r="${hand_radius}" l="${hand_length}"
+                                o_xyz="0 0 ${hand_length / 2.0}" o_rpy="0 0 0" />
     </link>
     <joint name="arm_joint1" type="revolute">
